File: nrw65-pcb/nrw65-pcb.kicad_pcb (KiCad board)
At the start: 2 copper layers, 122 parts, among them U1 nice_nano

Commit message: Work in progress
Parts:
- added BT1: Battery_Cell, Connector_JST:JST_PH_S2B-PH-K_1x02_P2.00mm_Horizontal, B.Cu at (144.2, 35.9)
- added SW1: SW_DIP_x01, Kicad footprints:MSK-12C02, F.Cu at (169.3, 38.1)
- added SW2: SW_DIP_x01, Connector_Wire:SolderWire-0.75sqmm_1x02_P7mm_D1.25mm_OD3.5mm, F.Cu at (156.4, 41.8)
- moved U1 187.0 mm to (103.8, 34.0), turned to 90 degrees
Connections:
- U1 pad 13: unconnected-(U1-BAT+-Pad13) -> bat
- U1 pad 14: unconnected-(U1-GND-Pad14) -> gnd
- U1 pad 15: unconnected-(U1-RST-Pad15) -> rst
- U1 pad 29: unconnected-(U1-BAT+-Pad29) -> bat
- U1 pad 3: unconnected-(U1-GND-Pad3) -> gnd
- U1 pad 4: unconnected-(U1-GND-Pad4) -> gnd

Commit message: add pcb and rcheme routing
Parts:
- SW1, SW2: moved to B.Cu
- moved U1 186.6 mm to (269.4, 120.0), turned to 180 degrees
- moved BT1 129.7 mm to (250.1, 110.7), turned to 90 degrees
- moved SW2 118.6 mm to (257.5, 103.8), turned to -90 degrees
- moved SW1 101.9 mm to (257.9, 88.5), turned to 90 degrees
- moved D59 1.77 mm to (258.7, 145.2)
Connections:
- D1 pad 1: Net-(D1-K) -> row0
- D10 pad 1: Net-(D1-K) -> row0
- D11 pad 1: Net-(D1-K) -> row0
- D12 pad 1: Net-(D1-K) -> row0
- D13 pad 1: Net-(D1-K) -> row0
- D14 pad 1: Net-(D14-K) -> row1
- D15 pad 1: Net-(D14-K) -> row1
- D16 pad 1: Net-(D14-K) -> row1
- D17 pad 1: Net-(D14-K) -> row1
- D18 pad 1: Net-(D14-K) -> row1
- D19 pad 1: Net-(D14-K) -> row1
- D2 pad 1: Net-(D1-K) -> row0
- D20 pad 1: Net-(D14-K) -> row1
- D21 pad 1: Net-(D14-K) -> row1
- D22 pad 1: Net-(D14-K) -> row1
- D23 pad 1: Net-(D14-K) -> row1
- D24 pad 1: Net-(D14-K) -> row1
- D25 pad 1: Net-(D14-K) -> row1
- D26 pad 1: Net-(D14-K) -> row1
- D27 pad 1: Net-(D27-K) -> row2
- D28 pad 1: Net-(D27-K) -> row2
- D29 pad 1: Net-(D27-K) -> row2
- D3 pad 1: Net-(D1-K) -> row0
- D30 pad 1: Net-(D27-K) -> row2
- D31 pad 1: Net-(D27-K) -> row2
- D32 pad 1: Net-(D27-K) -> row2
- D33 pad 1: Net-(D27-K) -> row2
- D34 pad 1: Net-(D27-K) -> row2
- D35 pad 1: Net-(D27-K) -> row2
- D36 pad 1: Net-(D27-K) -> row2
- D37 pad 1: Net-(D27-K) -> row2
- D38 pad 1: Net-(D27-K) -> row2
- D39 pad 1: Net-(D39-K) -> row3
- D4 pad 1: Net-(D1-K) -> row0
- D40 pad 1: Net-(D39-K) -> row3
- D41 pad 1: Net-(D39-K) -> row3
- D42 pad 1: Net-(D39-K) -> row3
- D43 pad 1: Net-(D39-K) -> row3
- D44 pad 1: Net-(D39-K) -> row3
- D45 pad 1: Net-(D39-K) -> row3
- D46 pad 1: Net-(D39-K) -> row3
- D47 pad 1: Net-(D39-K) -> row3
- D48 pad 1: Net-(D39-K) -> row3
- D49 pad 1: Net-(D39-K) -> row3
- D5 pad 1: Net-(D1-K) -> row0
- D50 pad 1: Net-(D39-K) -> row3
- D51 pad 1: Net-(D51-K) -> row4
- D52 pad 1: Net-(D51-K) -> row4
- D53 pad 1: Net-(D51-K) -> row4
- D54 pad 1: Net-(D51-K) -> row4
- D55 pad 1: Net-(D51-K) -> row4
- D56 pad 1: Net-(D51-K) -> row4
- D57 pad 1: Net-(D51-K) -> row4
- D58 pad 1: Net-(D51-K) -> row4
- D59 pad 1: Net-(D51-K) -> row4
- D6 pad 1: Net-(D1-K) -> row0
- D7 pad 1: Net-(D1-K) -> row0
- D8 pad 1: Net-(D1-K) -> row0
- D9 pad 1: Net-(D1-K) -> row0
- MX1 pad 1: Net-(MX1-Pad1) -> col0
- MX10 pad 1: Net-(MX10-Pad1) -> col9
- MX11 pad 1: Net-(MX11-Pad1) -> col10
- MX12 pad 1: Net-(MX12-Pad1) -> col11
- MX13 pad 1: Net-(MX13-Pad1) -> col12
- MX14 pad 1: Net-(MX1-Pad1) -> col0
- MX15 pad 1: Net-(MX15-Pad1) -> col1
- MX16 pad 1: Net-(MX16-Pad1) -> col2
- MX17 pad 1: Net-(MX17-Pad1) -> col3
- MX18 pad 1: Net-(MX18-Pad1) -> col4
- MX19 pad 1: Net-(MX19-Pad1) -> col5
- MX2 pad 1: Net-(MX15-Pad1) -> col1
- MX20 pad 1: Net-(MX20-Pad1) -> col6
- MX21 pad 1: Net-(MX21-Pad1) -> col7
- MX22 pad 1: Net-(MX22-Pad1) -> col8
- MX23 pad 1: Net-(MX10-Pad1) -> col9
- MX24 pad 1: Net-(MX11-Pad1) -> col10
- MX25 pad 1: Net-(MX12-Pad1) -> col11
- MX26 pad 1: Net-(MX13-Pad1) -> col12
- MX27 pad 1: Net-(MX1-Pad1) -> col0
- MX28 pad 1: Net-(MX15-Pad1) -> col1
- MX29 pad 1: Net-(MX16-Pad1) -> col2
- MX3 pad 1: Net-(MX16-Pad1) -> col2
- MX30 pad 1: Net-(MX17-Pad1) -> col3
- MX31 pad 1: Net-(MX18-Pad1) -> col4
- MX32 pad 1: Net-(MX19-Pad1) -> col5
- MX33 pad 1: Net-(MX20-Pad1) -> col6
- MX34 pad 1: Net-(MX21-Pad1) -> col7
- MX35 pad 1: Net-(MX22-Pad1) -> col8
- MX36 pad 1: Net-(MX10-Pad1) -> col9
- MX37 pad 1: Net-(MX11-Pad1) -> col10
- MX38 pad 1: Net-(MX13-Pad1) -> col12
- MX39 pad 1: Net-(MX1-Pad1) -> col0
- MX4 pad 1: Net-(MX17-Pad1) -> col3
- MX40 pad 1: Net-(MX15-Pad1) -> col1
- MX41 pad 1: Net-(MX16-Pad1) -> col2
- MX42 pad 1: Net-(MX17-Pad1) -> col3
- MX43 pad 1: Net-(MX18-Pad1) -> col4
- MX44 pad 1: Net-(MX19-Pad1) -> col5
- MX45 pad 1: Net-(MX20-Pad1) -> col6
- MX46 pad 1: Net-(MX21-Pad1) -> col7
- MX47 pad 1: Net-(MX22-Pad1) -> col8
- MX48 pad 1: Net-(MX10-Pad1) -> col9
- MX49 pad 1: Net-(MX11-Pad1) -> col10
- MX5 pad 1: Net-(MX18-Pad1) -> col4
- MX50 pad 1: Net-(MX12-Pad1) -> col11
- MX51 pad 1: Net-(MX1-Pad1) -> col0
- MX52 pad 1: Net-(MX15-Pad1) -> col1
- MX53 pad 1: Net-(MX16-Pad1) -> col2
- MX54 pad 1: Net-(MX10-Pad1) -> col9
- MX55 pad 1: Net-(MX18-Pad1) -> col4
- MX56 pad 1: Net-(MX21-Pad1) -> col7
- MX57 pad 1: Net-(MX11-Pad1) -> col10
- MX58 pad 1: Net-(MX12-Pad1) -> col11
- MX59 pad 1: Net-(MX13-Pad1) -> col12
- MX6 pad 1: Net-(MX19-Pad1) -> col5
- MX7 pad 1: Net-(MX20-Pad1) -> col6
- MX8 pad 1: Net-(MX21-Pad1) -> col7
- MX9 pad 1: Net-(MX22-Pad1) -> col8
- U1 pad 1: unconnected-(U1-P0.06-Pad1) -> row0
- U1 pad 10: unconnected-(U1-P0.11-Pad10) -> col4
- U1 pad 11: unconnected-(U1-P1.04-LF-Pad11) -> col3
- U1 pad 12: unconnected-(U1-P1.06-LF-Pad12) -> row4
- U1 pad 17: unconnected-(U1-P0.31-LF-Pad17) -> col11
- U1 pad 18: unconnected-(U1-P0.29-LF-Pad18) -> col0
- U1 pad 19: unconnected-(U1-P0.02-LF-Pad19) -> col1
- U1 pad 2: unconnected-(U1-P0.08-Pad2) -> row1
- U1 pad 20: unconnected-(U1-P1.15-LF-Pad20) -> col2
- U1 pad 21: unconnected-(U1-P1.13-LF-Pad21) -> row3
- U1 pad 22: unconnected-(U1-P1.11-LF-Pad22) -> col7
- U1 pad 23: unconnected-(U1-P0-10-LF-Pad23) -> col9
- U1 pad 24: unconnected-(U1-P0.09-LF-Pad24) -> col10
- U1 pad 28: unconnected-(U1-GND-Pad28) -> gnd
- U1 pad 5: unconnected-(U1-P0.17-Pad5) -> row2
- U1 pad 6: unconnected-(U1-P0.20-Pad6) -> col12
- U1 pad 7: unconnected-(U1-P0.22-Pad7) -> col8
- U1 pad 8: unconnected-(U1-P0.24-Pad8) -> col6
- U1 pad 9: unconnected-(U1-P1.00-Pad9) -> col5
Routing:
- net col2: track 0.00 -> 361.4 mm
- net col1: track 0.00 -> 343.3 mm
- net col0: track 0.00 -> 331.1 mm
- net row0: track 0.00 -> 293.0 mm
- net row2: track 0.00 -> 290.4 mm
- net row1: track 0.00 -> 283.8 mm
- net col3: track 0.00 -> 276.3 mm
- net col4: track 0.00 -> 274.0 mm
- net row4: track 0.00 -> 262.1 mm
- net col5: track 0.00 -> 248.8 mm
- net col6: track 0.00 -> 233.4 mm
- net row3: track 0.00 -> 229.8 mm
- net col7: track 0.00 -> 201.1 mm
- net col8: track 0.00 -> 195.3 mm
- net col9: track 0.00 -> 158.9 mm
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
Commit message: Work in progress: change to Pro Micro footprint, add rotary encoder, change to MX+KS33 hot swap footprints, reroute tracks.
Parts:
- removed SW2: SW_DIP_x01, Connector_Wire:SolderWire-0.75sqmm_1x02_P7mm_D1.25mm_OD3.5mm
- added G***: LOGO, nrw65-pcb:monogorod, F.Cu at (157.7, 78.8)
- MX1, MX10, MX11, MX14, MX15, MX16, MX17, MX18, MX19, MX2, MX20, MX21, MX22, MX23, MX24, MX25, MX26, MX28, MX29, MX3, MX30, MX31, MX32, MX33, MX34, MX35, MX36, MX37, MX38, MX4, MX40, MX41, MX42, MX43, MX44, MX45, MX46, MX47, MX48, MX49, MX5, MX50, MX55, MX56, MX57, MX58, MX59, MX6, MX7, MX8, MX9: footprint PCM_marbastlib-mx:SW_MX_HS_S_1u_REVERSE -> PCM_marbastlib-mx:SW_MX_HS_S_1u_REVERSE+KS33_HS
- MX12: footprint PCM_marbastlib-mx:SW_MX_HS_S_1u_REVERSE -> PCM_marbastlib-mx:SW_MX_1u+KS33
- MX13: value MX_SW_HS -> RotaryEncoder_Switch; footprint PCM_marbastlib-mx:SW_MX_HS_S_1u_REVERSE -> PCM_marbastlib-various:ROT_Alps_EC11E-Switch_Invisible_designator
- MX27, MX51, MX52, MX53, MX54: footprint PCM_marbastlib-mx:SW_MX_HS_S_1.25u_REVERSE -> PCM_marbastlib-mx:SW_MX_HS_S_1.25u_REVERSE+KS33_HS
- MX39: footprint PCM_marbastlib-mx:SW_MX_HS_S_1.5u_REVERSE -> PCM_marbastlib-mx:SW_MX_HS_S_1.5u_REVERSE+KS33_HS
- U1: value nice_nano -> ProMicro; footprint PCM_marbastlib-xp-promicroish:nice_nano_AH_USBup -> PCM_marbastlib-xp-promicroish:ProMicro_USBup
- moved U1 85.4 mm to (267.9, 34.6), turned to 90 degrees
- moved BT1 61.9 mm to (257.2, 49.2)
- moved SW1 40.7 mm to (265.3, 48.5)
- moved D59 36.6 mm to (285.9, 120.7)
- moved D14 27.9 mm to (43.0, 58.8)
- moved D15 27.9 mm to (62.0, 58.8)
- moved D16 27.9 mm to (81.1, 58.8)
- moved D17 27.9 mm to (100.2, 58.8)
- moved D18 27.9 mm to (119.2, 58.8)
- moved D19 27.9 mm to (138.2, 58.8)
- moved D20 27.9 mm to (157.3, 58.8)
- moved D21 27.9 mm to (176.3, 58.8)
- moved D22 27.9 mm to (195.4, 58.8)
- moved D23 27.9 mm to (214.4, 58.8)
- moved D24 27.9 mm to (233.5, 58.8)
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Connections:
- D11 pad 1: row0 -> row5
- D12 pad 1: row0 -> row5
- D13 pad 1: row0 -> row5
- D24 pad 1: row1 -> row5
- D25 pad 1: row1 -> row5
- D26 pad 1: row1 -> row5
- D37 pad 1: row2 -> row5
- D38 pad 1: row2 -> row5
- D49 pad 1: row3 -> row5
- D50 pad 1: row3 -> row4
- MX11 pad 1: col10 -> col2
- MX12 pad 1: col11 -> col1
- MX24 pad 1: col10 -> col5
- MX25 pad 1: col11 -> col4
- MX26 pad 1: col12 -> col3
- MX37 pad 1: col10 -> col8
- MX38 pad 1: col12 -> col7
- MX49 pad 1: col10 -> col6
- MX50 pad 1: col11 -> col9
- MX54 pad 1: col9 -> col5
- MX55 pad 1: col4 -> col3
- MX56 pad 1: col7 -> col4
- MX57 pad 1: col10 -> col6
- MX58 pad 1: col11 -> col7
- MX59 pad 1: col12 -> col8
- SW1 pad 2: bat -> raw
- U1 pad 1: row0 -> row4
- U1 pad 11: col3 -> col2
- U1 pad 12: row4 -> col1
- U1 pad 13: bat -> raw
- U1 pad 16: unconnected-(U1-3V3-Pad16) -> vcc
- U1 pad 17: col11 -> rotB
- U1 pad 18: col0 -> rotA
- U1 pad 19: col1 -> col0
- U1 pad 2: row1 -> col3
- U1 pad 20: col2 -> row5
- U1 pad 21: row3 -> row0
- U1 pad 22: col7 -> row1
- U1 pad 23: col9 -> row2
- U1 pad 24: col10 -> row3
- U1 pad 5: row2 -> col7
- U1 pad 6: col12 -> col8
- U1 pad 7: col8 -> col9
Routing:
- net row5: track 0.00 -> 210.4 mm
- net col10: track 138.5 -> 0.00 mm
- net col5: track 248.8 -> 380.1 mm
- net row4: track 262.1 -> 387.5 mm
- net col8: track 195.3 -> 312.6 mm
- net col11: track 109.7 -> 0.00 mm
- net row3: track 229.8 -> 335.8 mm, vias 0 -> 2
- net col12: track 97.1 -> 0.00 mm
- net col7: track 201.1 -> 291.8 mm
- net col4: track 274.0 -> 341.9 mm
- net col3: track 276.3 -> 342.0 mm, vias 0 -> 1
- net col6: track 233.4 -> 296.0 mm, vias 0 -> 2
- net col2: track 361.4 -> 300.7 mm
- net col9: track 158.9 -> 203.0 mm, vias 0 -> 1
- net raw: track 0.00 -> 33.9 mm
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Other:
- board outline added: 271.9 x 112.2 mm

Commit message: Work in progress
Parts:
- turned S55 to 180 degrees
- turned S56 to 180 degrees
Routing:
- net row4: track 387.5 -> 389.6 mm
- net col4: track 341.9 -> 343.1 mm
- net col8: track 312.6 -> 313.6 mm
- net col6: track 296.0 -> 296.7 mm
Other:
- board size 271.9 x 112.2 mm -> 275.9 x 118.8 mm
